Commit message: add loaded robots and forklift

File: turtlebot3/turtlebot3_description/urdf/turtlebot3_waffle.gazebo.xacro (robot description, xacro)
@@ -102,5 +102,5 @@
     </plugin>
   </gazebo>
-  <gazebo reference="base_scan">
+  <!-- <gazebo reference="base_scan">
     <material>Gazebo/FlatBlack</material>
     <sensor type="ray" name="lds_lfcd_sensor">
@@ -176,4 +176,4 @@
       </plugin>
     </sensor>
-  </gazebo>
+  </gazebo> -->
 </robot>

File: turtlebot3/turtlebot3_description/urdf/turtlebot3_waffle.urdf.xacro (robot description, xacro)
@@ -137,10 +137,10 @@
   </joint>
   <link name="imu_link"/>
-  <joint name="scan_joint" type="fixed">
+  <!-- <joint name="scan_joint" type="fixed">
     <parent link="base_link"/>
     <child link="base_scan"/>
     <origin xyz="-0.064 0 0.122" rpy="0 0 0"/>
-  </joint>
-  <link name="base_scan">
+  </joint> -->
+  <!-- <link name="base_scan">
     <visual>
       <origin xyz="0 0 0" rpy="0 0 0"/>
@@ -163,6 +163,6 @@
                izz="0.001" />
     </inertial>
-  </link>
-  <joint name="camera_joint" type="fixed">
+  </link> -->
+  <!-- <joint name="camera_joint" type="fixed">
     <origin xyz="0.064 -0.065 0.094" rpy="0 0 0"/>
     <parent link="base_link"/>
@@ -181,5 +181,5 @@
         <box size="0.012 0.132 0.020"/>
       </geometry>
-    </collision>
+    </collision> -->
     <!-- This inertial field needs doesn't contain reliable data!! -->
 <!--   <inertial>
@@ -190,5 +190,5 @@
                izz="0.003879257" />
     </inertial>-->
-  </link>
+  <!-- </link>
   <joint name="camera_rgb_joint" type="fixed">
     <origin xyz="${r200_cam_rgb_px} ${r200_cam_rgb_py} ${r200_cam_rgb_pz}" rpy="0 0 0"/>
@@ -214,4 +214,4 @@
     <child link="camera_depth_optical_frame"/>
   </joint>
-  <link name="camera_depth_optical_frame"/>
+  <link name="camera_depth_optical_frame"/> -->
 </robot>

File: velodyne_simulator/velodyne_description/urdf/velodyne.urdf.xacro (robot description, xacro)
@@ -27,7 +27,5 @@
       <origin xyz="0 0 0"/>
       <mass value="10"/>
-      <inertia ixx="3.0" ixy="0.0" ixz="0.0"
-               iyy="3.0" iyz="0.0"
-               izz="3.0" />
+        <inertia ixx="0.01" ixy="0" ixz="0" iyy="0.01" iyz="0" izz="0.01" />
     </inertial>
   </link>

File: velodyne_simulator/velodyne_description/urdf/velodyne_warehouse.urdf.xacro (robot description, xacro)
@@ -11,5 +11,5 @@
    <parent link="base_footprint" />
     <child link="base_link" />
-    <origin xyz="0 0 0.05" rpy="0 0 0" />
+    <origin xyz="0 0 0.03" rpy="0 0 0" />
   </joint>
   <link name="base_link" >
@@ -27,7 +27,5 @@
       <origin xyz="0 0 0"/>
       <mass value="10"/>
-      <inertia ixx="3.0" ixy="0.0" ixz="0.0"
-               iyy="3.0" iyz="0.0"
-               izz="3.0" />
+      <inertia ixx="0.01" ixy="0" ixz="0" iyy="0.01" iyz="0" izz="0.01" />
     </inertial>
   </link>
