Commit message: edit forklift.urdf.xacro

File: turtlebot3/turtlebot3_description/urdf/turtlebot3_forklift.urdf.xacro (robot description, xacro)
@@ -20,5 +20,5 @@
       <origin xyz="0 0 0.070" rpy="0 0 0"/>
       <geometry>
-       <mesh filename="package://turtlebot3_description/meshes/bases/forklift_base_convex.dae"  />
+        <mesh filename="package://turtlebot3_description/meshes/bases/forklift_base.STL" scale="3.0 3.0 3.0"/>
       </geometry>
     </collision>

File: turtlebot3/turtlebot3_description/urdf/turtlebot3_forklift_w_load.urdf.xacro (robot description, xacro)
@@ -20,5 +20,5 @@
       <origin xyz="0 0 0.070" rpy="0 0 0"/>
       <geometry>
-       <mesh filename="package://turtlebot3_description/meshes/bases/forklift_base_convex.dae"  />
+        <mesh filename="package://turtlebot3_description/meshes/bases/forklift_base_w_load.STL" scale="0.3 0.3 0.3"/>
       </geometry>
     </collision>
