Commit message: edit .urdf.xacro files to correct size shown in rviz

File: turtlebot3/turtlebot3_description/urdf/amr.urdf.xacro (robot description, xacro)
@@ -13,12 +13,12 @@
       <origin xyz="-0.032 0 0.0" rpy="0 0 0"/>
       <geometry>
-        <mesh filename="package://turtlebot3_description/meshes/bases/robot_base.dae" scale="0.5 0.5 0.7"/>
+        <mesh filename="package://turtlebot3_description/meshes/bases/robot_base.dae" scale="0.5 0.5 0.3"/>
       </geometry>
       <material name="light_black"/>
     </visual>
     <collision>
-      <origin xyz="-0.032 0 0.070" rpy="0 0 0"/>
+      <origin xyz="-0.032 0 0.250" rpy="0 0 0"/>
       <geometry>
-        <box size="0.140 0.140 0.143"/>
+        <mesh filename="package://turtlebot3_description/meshes/bases/robot_base.dae" scale="0.5 0.7 0.3"/>
       </geometry>
     </collision>
@@ -34,5 +34,5 @@
     <parent link="base_link_burger"/>
     <child link="wheel_left_link"/>
-    <origin xyz="0.0 0.08 0.023" rpy="-1.57 0 0"/>
+    <origin xyz="0.0 0.2 0.023" rpy="-1.57 0 0"/>
     <axis xyz="0 0 1"/>
   </joint>
@@ -62,5 +62,5 @@
     <parent link="base_link_burger"/>
     <child link="wheel_right_link"/>
-    <origin xyz="0.0 -0.080 0.023" rpy="-1.57 0 0"/>
+    <origin xyz="0.0 -0.2 0.023" rpy="-1.57 0 0"/>
     <axis xyz="0 0 1"/>
   </joint>

File: turtlebot3/turtlebot3_description/urdf/amr_w_load.urdf.xacro (robot description, xacro)
@@ -18,7 +18,7 @@
     </visual>
     <collision>
-      <origin xyz="-0.032 0 0.070" rpy="0 0 0"/>
+      <origin xyz="-0.032 0 0.250" rpy="0 0 0"/>
       <geometry>
-        <box size="0.140 0.140 0.143"/>
+        <mesh filename="package://turtlebot3_description/meshes/bases/robot_base_w_load.dae" scale="0.5 0.7 0.7"/>
       </geometry>
     </collision>
@@ -34,5 +34,5 @@
     <parent link="base_link_burger"/>
     <child link="wheel_left_link"/>
-    <origin xyz="0.0 0.08 0.023" rpy="-1.57 0 0"/>
+    <origin xyz="0.0 0.2 0.023" rpy="-1.57 0 0"/>
     <axis xyz="0 0 1"/>
   </joint>
@@ -62,5 +62,5 @@
     <parent link="base_link_burger"/>
     <child link="wheel_right_link"/>
-    <origin xyz="0.0 -0.080 0.023" rpy="-1.57 0 0"/>
+    <origin xyz="0.0 -0.2 0.023" rpy="-1.57 0 0"/>
     <axis xyz="0 0 1"/>
   </joint>

File: turtlebot3/turtlebot3_description/urdf/rectangle_amr.urdf.xacro (robot description, xacro)
@@ -13,12 +13,12 @@
       <origin xyz="-0.032 0 0.0" rpy="0 0 0"/>
       <geometry>
-        <mesh filename="package://turtlebot3_description/meshes/bases/robot_base.dae" scale="0.5 0.7 0.7"/>
+        <mesh filename="package://turtlebot3_description/meshes/bases/robot_base.dae" scale="0.5 0.7 0.3"/>
       </geometry>
       <material name="light_black"/>
     </visual>
     <collision>
-      <origin xyz="-0.032 0 0.070" rpy="0 0 0"/>
+      <origin xyz="-0.032 0 0.250" rpy="0 0 0"/>
       <geometry>
-        <box size="0.140 0.140 0.143"/>
+        <mesh filename="package://turtlebot3_description/meshes/bases/robot_base.dae" scale="0.5 0.7 0.3"/>
       </geometry>
     </collision>
@@ -34,5 +34,5 @@
     <parent link="base_link_burger"/>
     <child link="wheel_left_link"/>
-    <origin xyz="0.0 0.08 0.023" rpy="-1.57 0 0"/>
+    <origin xyz="0.0 0.2 0.023" rpy="-1.57 0 0"/>
     <axis xyz="0 0 1"/>
   </joint>
@@ -62,5 +62,5 @@
     <parent link="base_link_burger"/>
     <child link="wheel_right_link"/>
-    <origin xyz="0.0 -0.080 0.023" rpy="-1.57 0 0"/>
+    <origin xyz="0.0 -0.20 0.023" rpy="-1.57 0 0"/>
     <axis xyz="0 0 1"/>
   </joint>

File: turtlebot3/turtlebot3_description/urdf/rectangle_amr_w_load.urdf.xacro (robot description, xacro)
@@ -18,7 +18,7 @@
     </visual>
     <collision>
-      <origin xyz="-0.032 0 0.070" rpy="0 0 0"/>
+      <origin xyz="-0.032 0 0.250" rpy="0 0 0"/>
       <geometry>
-        <box size="0.140 0.140 0.143"/>
+        <mesh filename="package://turtlebot3_description/meshes/bases/robot_base_w_load.dae" scale="0.5 0.7 0.7"/>
       </geometry>
     </collision>
@@ -34,5 +34,5 @@
     <parent link="base_link_burger"/>
     <child link="wheel_left_link"/>
-    <origin xyz="0.0 0.08 0.023" rpy="-1.57 0 0"/>
+    <origin xyz="0.0 0.2 0.023" rpy="-1.57 0 0"/>
     <axis xyz="0 0 1"/>
   </joint>
@@ -62,5 +62,5 @@
     <parent link="base_link_burger"/>
     <child link="wheel_right_link"/>
-    <origin xyz="0.0 -0.080 0.023" rpy="-1.57 0 0"/>
+    <origin xyz="0.0 -0.2 0.023" rpy="-1.57 0 0"/>
     <axis xyz="0 0 1"/>
   </joint>
