Commit message: clear miscellaneous

File: turtlebot3/turtlebot3_description/urdf/amr.urdf.xacro (robot description, xacro)
@@ -1,13 +1,13 @@
 <?xml version="1.0" ?>
-<robot name="turtlebot3_burger" xmlns:xacro="http://ros.org/wiki/xacro">
+<robot name="amr" xmlns:xacro="http://ros.org/wiki/xacro">
   <xacro:include filename="$(find turtlebot3_description)/urdf/common_properties.xacro"/>
-  <xacro:include filename="$(find turtlebot3_description)/urdf/turtlebot3_burger.gazebo.xacro"/>
-  <link name="base_footprint_burger"/>
-  <joint name="base_joint_burger" type="fixed">
-    <parent link="base_footprint_burger"/>
-    <child link="base_link_burger"/>
+  <xacro:include filename="$(find turtlebot3_description)/urdf/amr.gazebo.xacro"/>
+  <link name="base_footprint"/>
+  <joint name="base_joint" type="fixed">
+    <parent link="base_footprint"/>
+    <child link="base_link"/>
     <origin xyz="0.0 0.0 0.10" rpy="0 0 0"/>
   </joint>
-  <link name="base_link_burger">
+  <link name="base_link">
     <visual>
       <origin xyz="-0.032 0 0.0" rpy="0 0 0"/>
@@ -32,5 +32,5 @@
   </link>
   <joint name="wheel_left_joint" type="continuous">
-    <parent link="base_link_burger"/>
+    <parent link="base_link"/>
     <child link="wheel_left_link"/>
     <origin xyz="0.0 0.2 0.023" rpy="-1.57 0 0"/>
@@ -60,5 +60,5 @@
   </link>
   <joint name="wheel_right_joint" type="continuous">
-    <parent link="base_link_burger"/>
+    <parent link="base_link"/>
     <child link="wheel_right_link"/>
     <origin xyz="0.0 -0.2 0.023" rpy="-1.57 0 0"/>
@@ -88,5 +88,5 @@
   </link>
   <joint name="caster_back_joint" type="fixed">
-    <parent link="base_link_burger"/>
+    <parent link="base_link"/>
     <child link="caster_back_link"/>
     <origin xyz="-0.081 0 -0.004" rpy="-1.57 0 0"/>
@@ -108,35 +108,8 @@
   </link>
   <joint name="imu_joint" type="fixed">
-    <parent link="base_link_burger"/>
+    <parent link="base_link"/>
     <child link="imu_link"/>
     <origin xyz="-0.032 0 0.068" rpy="0 0 0"/>
   </joint>
   <link name="imu_link"/>
-  <!-- <joint name="scan_joint" type="fixed">
-    <parent link="base_link_burger"/>
-    <child link="base_scan"/>
-    <origin xyz="-0.032 0 0.172" rpy="0 0 0"/>
-  </joint>
-  <link name="base_scan">
-    <visual>
-      <origin xyz="0 0 0.0" rpy="0 0 0"/>
-      <geometry>
-        <mesh filename="package://turtlebot3_description/meshes/sensors/lds.stl" scale="0.001 0.001 0.001"/>
-      </geometry>
-      <material name="dark"/>
-    </visual>
-    <collision>
-      <origin xyz="0.015 0 -0.0065" rpy="0 0 0"/>
-      <geometry>
-        <cylinder length="0.0315" radius="0.055"/>
-      </geometry>
-    </collision>
-    <inertial>
-      <mass value="0.114" />
-      <origin xyz="0 0 0" />
-      <inertia ixx="0.001" ixy="0.0" ixz="0.0"
-               iyy="0.001" iyz="0.0"
-               izz="0.001" />
-    </inertial>
-  </link> -->
 </robot>

File: turtlebot3/turtlebot3_description/urdf/amr_w_load.urdf.xacro (robot description, xacro)
@@ -1,13 +1,13 @@
 <?xml version="1.0" ?>
-<robot name="turtlebot3_burger" xmlns:xacro="http://ros.org/wiki/xacro">
+<robot name="amr_w_load" xmlns:xacro="http://ros.org/wiki/xacro">
   <xacro:include filename="$(find turtlebot3_description)/urdf/common_properties.xacro"/>
-  <xacro:include filename="$(find turtlebot3_description)/urdf/turtlebot3_burger.gazebo.xacro"/>
-  <link name="base_footprint_burger"/>
-  <joint name="base_joint_burger" type="fixed">
-    <parent link="base_footprint_burger"/>
-    <child link="base_link_burger"/>
+  <xacro:include filename="$(find turtlebot3_description)/urdf/amr.gazebo.xacro"/>
+  <link name="base_footprint"/>
+  <joint name="base_joint" type="fixed">
+    <parent link="base_footprint"/>
+    <child link="base_link"/>
     <origin xyz="0.0 0.0 0.10" rpy="0 0 0"/>
   </joint>
-  <link name="base_link_burger">
+  <link name="base_link">
     <visual>
       <origin xyz="-0.032 0 0.0" rpy="0 0 0"/>
@@ -32,5 +32,5 @@
   </link>
   <joint name="wheel_left_joint" type="continuous">
-    <parent link="base_link_burger"/>
+    <parent link="base_link"/>
     <child link="wheel_left_link"/>
     <origin xyz="0.0 0.2 0.023" rpy="-1.57 0 0"/>
@@ -60,5 +60,5 @@
   </link>
   <joint name="wheel_right_joint" type="continuous">
-    <parent link="base_link_burger"/>
+    <parent link="base_link"/>
     <child link="wheel_right_link"/>
     <origin xyz="0.0 -0.2 0.023" rpy="-1.57 0 0"/>
@@ -88,5 +88,5 @@
   </link>
   <joint name="caster_back_joint" type="fixed">
-    <parent link="base_link_burger"/>
+    <parent link="base_link"/>
     <child link="caster_back_link"/>
     <origin xyz="-0.081 0 -0.004" rpy="-1.57 0 0"/>
@@ -108,35 +108,8 @@
   </link>
   <joint name="imu_joint" type="fixed">
-    <parent link="base_link_burger"/>
+    <parent link="base_link"/>
     <child link="imu_link"/>
     <origin xyz="-0.032 0 0.068" rpy="0 0 0"/>
   </joint>
   <link name="imu_link"/>
-  <!-- <joint name="scan_joint" type="fixed">
-    <parent link="base_link_burger"/>
-    <child link="base_scan"/>
-    <origin xyz="-0.032 0 0.172" rpy="0 0 0"/>
-  </joint>
-  <link name="base_scan">
-    <visual>
-      <origin xyz="0 0 0.0" rpy="0 0 0"/>
-      <geometry>
-        <mesh filename="package://turtlebot3_description/meshes/sensors/lds.stl" scale="0.001 0.001 0.001"/>
-      </geometry>
-      <material name="dark"/>
-    </visual>
-    <collision>
-      <origin xyz="0.015 0 -0.0065" rpy="0 0 0"/>
-      <geometry>
-        <cylinder length="0.0315" radius="0.055"/>
-      </geometry>
-    </collision>
-    <inertial>
-      <mass value="0.114" />
-      <origin xyz="0 0 0" />
-      <inertia ixx="0.001" ixy="0.0" ixz="0.0"
-               iyy="0.001" iyz="0.0"
-               izz="0.001" />
-    </inertial>
-  </link> -->
 </robot>

File: turtlebot3/turtlebot3_description/urdf/rectangle_amr.urdf.xacro (robot description, xacro)
@@ -1,13 +1,13 @@
 <?xml version="1.0" ?>
-<robot name="turtlebot3_burger" xmlns:xacro="http://ros.org/wiki/xacro">
+<robot name="rectangle_amr" xmlns:xacro="http://ros.org/wiki/xacro">
   <xacro:include filename="$(find turtlebot3_description)/urdf/common_properties.xacro"/>
-  <xacro:include filename="$(find turtlebot3_description)/urdf/turtlebot3_burger.gazebo.xacro"/>
-  <link name="base_footprint_burger"/>
-  <joint name="base_joint_burger" type="fixed">
-    <parent link="base_footprint_burger"/>
-    <child link="base_link_burger"/>
+  <xacro:include filename="$(find turtlebot3_description)/urdf/amr.gazebo.xacro"/>
+  <link name="base_footprint"/>
+  <joint name="base_joint" type="fixed">
+    <parent link="base_footprint"/>
+    <child link="base_link"/>
     <origin xyz="0.0 0.0 0.10" rpy="0 0 0"/>
   </joint>
-  <link name="base_link_burger">
+  <link name="base_link">
     <visual>
       <origin xyz="-0.032 0 0.0" rpy="0 0 0"/>
@@ -32,5 +32,5 @@
   </link>
   <joint name="wheel_left_joint" type="continuous">
-    <parent link="base_link_burger"/>
+    <parent link="base_link"/>
     <child link="wheel_left_link"/>
     <origin xyz="0.0 0.2 0.023" rpy="-1.57 0 0"/>
@@ -60,5 +60,5 @@
   </link>
   <joint name="wheel_right_joint" type="continuous">
-    <parent link="base_link_burger"/>
+    <parent link="base_link"/>
     <child link="wheel_right_link"/>
     <origin xyz="0.0 -0.20 0.023" rpy="-1.57 0 0"/>
@@ -88,5 +88,5 @@
   </link>
   <joint name="caster_back_joint" type="fixed">
-    <parent link="base_link_burger"/>
+    <parent link="base_link"/>
     <child link="caster_back_link"/>
     <origin xyz="-0.081 0 -0.004" rpy="-1.57 0 0"/>
@@ -108,35 +108,8 @@
   </link>
   <joint name="imu_joint" type="fixed">
-    <parent link="base_link_burger"/>
+    <parent link="base_link"/>
     <child link="imu_link"/>
     <origin xyz="-0.032 0 0.068" rpy="0 0 0"/>
   </joint>
   <link name="imu_link"/>
-  <!-- <joint name="scan_joint" type="fixed">
-    <parent link="base_link_burger"/>
-    <child link="base_scan"/>
-    <origin xyz="-0.032 0 0.172" rpy="0 0 0"/>
-  </joint>
-  <link name="base_scan">
-    <visual>
-      <origin xyz="0 0 0.0" rpy="0 0 0"/>
-      <geometry>
-        <mesh filename="package://turtlebot3_description/meshes/sensors/lds.stl" scale="0.001 0.001 0.001"/>
-      </geometry>
-      <material name="dark"/>
-    </visual>
-    <collision>
-      <origin xyz="0.015 0 -0.0065" rpy="0 0 0"/>
-      <geometry>
-        <cylinder length="0.0315" radius="0.055"/>
-      </geometry>
-    </collision>
-    <inertial>
-      <mass value="0.114" />
-      <origin xyz="0 0 0" />
-      <inertia ixx="0.001" ixy="0.0" ixz="0.0"
-               iyy="0.001" iyz="0.0"
-               izz="0.001" />
-    </inertial>
-  </link> -->
 </robot>

File: turtlebot3/turtlebot3_description/urdf/rectangle_amr_w_load.urdf.xacro (robot description, xacro)
@@ -1,13 +1,13 @@
 <?xml version="1.0" ?>
-<robot name="turtlebot3_burger" xmlns:xacro="http://ros.org/wiki/xacro">
+<robot name="rectangle_amr_w_load" xmlns:xacro="http://ros.org/wiki/xacro">
   <xacro:include filename="$(find turtlebot3_description)/urdf/common_properties.xacro"/>
-  <xacro:include filename="$(find turtlebot3_description)/urdf/turtlebot3_burger.gazebo.xacro"/>
-  <link name="base_footprint_burger"/>
-  <joint name="base_joint_burger" type="fixed">
-    <parent link="base_footprint_burger"/>
-    <child link="base_link_burger"/>
+  <xacro:include filename="$(find turtlebot3_description)/urdf/amr.gazebo.xacro"/>
+  <link name="base_footprint"/>
+  <joint name="base_joint" type="fixed">
+    <parent link="base_footprint"/>
+    <child link="base_link"/>
     <origin xyz="0.0 0.0 0.10" rpy="0 0 0"/>
   </joint>
-  <link name="base_link_burger">
+  <link name="base_link">
     <visual>
       <origin xyz="-0.032 0 0.0" rpy="0 0 0"/>
@@ -32,5 +32,5 @@
   </link>
   <joint name="wheel_left_joint" type="continuous">
-    <parent link="base_link_burger"/>
+    <parent link="base_link"/>
     <child link="wheel_left_link"/>
     <origin xyz="0.0 0.2 0.023" rpy="-1.57 0 0"/>
@@ -60,5 +60,5 @@
   </link>
   <joint name="wheel_right_joint" type="continuous">
-    <parent link="base_link_burger"/>
+    <parent link="base_link"/>
     <child link="wheel_right_link"/>
     <origin xyz="0.0 -0.2 0.023" rpy="-1.57 0 0"/>
@@ -88,5 +88,5 @@
   </link>
   <joint name="caster_back_joint" type="fixed">
-    <parent link="base_link_burger"/>
+    <parent link="base_link"/>
     <child link="caster_back_link"/>
     <origin xyz="-0.081 0 -0.004" rpy="-1.57 0 0"/>
@@ -108,35 +108,8 @@
   </link>
   <joint name="imu_joint" type="fixed">
-    <parent link="base_link_burger"/>
+    <parent link="base_link"/>
     <child link="imu_link"/>
     <origin xyz="-0.032 0 0.068" rpy="0 0 0"/>
   </joint>
   <link name="imu_link"/>
-  <!-- <joint name="scan_joint" type="fixed">
-    <parent link="base_link_burger"/>
-    <child link="base_scan"/>
-    <origin xyz="-0.032 0 0.172" rpy="0 0 0"/>
-  </joint>
-  <link name="base_scan">
-    <visual>
-      <origin xyz="0 0 0.0" rpy="0 0 0"/>
-      <geometry>
-        <mesh filename="package://turtlebot3_description/meshes/sensors/lds.stl" scale="0.001 0.001 0.001"/>
-      </geometry>
-      <material name="dark"/>
-    </visual>
-    <collision>
-      <origin xyz="0.015 0 -0.0065" rpy="0 0 0"/>
-      <geometry>
-        <cylinder length="0.0315" radius="0.055"/>
-      </geometry>
-    </collision>
-    <inertial>
-      <mass value="0.114" />
-      <origin xyz="0 0 0" />
-      <inertia ixx="0.001" ixy="0.0" ixz="0.0"
-               iyy="0.001" iyz="0.0"
-               izz="0.001" />
-    </inertial>
-  </link> -->
 </robot>

File: turtlebot3/turtlebot3_description/urdf/turtlebot3_burger.urdf.xacro (robot description, xacro)
@@ -113,5 +113,5 @@
   </joint>
   <link name="imu_link"/>
-  <!-- <joint name="scan_joint" type="fixed">
+  <joint name="scan_joint" type="fixed">
     <parent link="base_link_burger"/>
     <child link="base_scan"/>
@@ -139,4 +139,4 @@
                izz="0.001" />
     </inertial>
-  </link> -->
+  </link>
 </robot>

File: turtlebot3/turtlebot3_description/urdf/turtlebot3_burger_w_load.gazebo.xacro (robot description, xacro)
@@ -1,7 +1,7 @@
 <?xml version="1.0"?>
-<robot name="amr_sim" xmlns:xacro="http://ros.org/wiki/xacro">
+<robot name="turtlebot3_burger_sim" xmlns:xacro="http://ros.org/wiki/xacro">
   <xacro:arg name="laser_visual" default="false"/>
   <xacro:arg name="imu_visual"   default="false"/>
-  <gazebo reference="base_link">
+  <gazebo reference="base_link_burger">
     <material>Gazebo/DarkGrey</material>
   </gazebo>
@@ -43,5 +43,5 @@
   </gazebo>
   <gazebo>
-    <plugin name="turtlebot3_controller" filename="libgazebo_ros_diff_drive.so">
+    <plugin name="turtlebot3_burger_controller" filename="libgazebo_ros_diff_drive.so">
       <commandTopic>cmd_vel</commandTopic>
       <odometryTopic>odom</odometryTopic>
@@ -49,5 +49,5 @@
       <odometrySource>world</odometrySource>
       <publishOdomTF>true</publishOdomTF>
-      <robotBaseFrame>base_footprint</robotBaseFrame>
+      <robotBaseFrame>base_footprint_burger</robotBaseFrame>
       <publishWheelTF>false</publishWheelTF>
       <publishTf>true</publishTf>
@@ -92,3 +92,35 @@
     </plugin>
   </gazebo>
+  <!-- <gazebo reference="base_scan">
+    <material>Gazebo/FlatBlack</material>
+    <sensor type="ray" name="lds_lfcd_sensor">
+      <pose>0 0 0 0 0 0</pose>
+      <visualize>$(arg laser_visual)</visualize>
+      <update_rate>5</update_rate>
+      <ray>
+        <scan>
+          <horizontal>
+            <samples>360</samples>
+            <resolution>1</resolution>
+            <min_angle>0.0</min_angle>
+            <max_angle>6.28319</max_angle>
+          </horizontal>
+        </scan>
+        <range>
+          <min>0.120</min>
+          <max>3.5</max>
+          <resolution>0.015</resolution>
+        </range>
+        <noise>
+          <type>gaussian</type>
+          <mean>0.0</mean>
+          <stddev>0.01</stddev>
+        </noise>
+      </ray>
+      <plugin name="gazebo_ros_lds_lfcd_controller" filename="libgazebo_ros_laser.so">
+        <topicName>scan</topicName>
+        <frameName>base_scan</frameName>
+      </plugin>
+    </sensor>
+  </gazebo> -->
 </robot>

File: turtlebot3/turtlebot3_description/urdf/turtlebot3_burger_w_load.urdf.xacro (robot description, xacro)
@@ -2,5 +2,5 @@
 <robot name="turtlebot3_burger" xmlns:xacro="http://ros.org/wiki/xacro">
   <xacro:include filename="$(find turtlebot3_description)/urdf/common_properties.xacro"/>
-  <xacro:include filename="$(find turtlebot3_description)/urdf/turtlebot3_burger.gazebo.xacro"/>
+  <xacro:include filename="$(find turtlebot3_description)/urdf/turtlebot3_burger_w_load.gazebo.xacro"/>
   <link name="base_footprint_burger"/>
   <joint name="base_joint_burger" type="fixed">
@@ -139,4 +139,4 @@
                izz="0.001" />
     </inertial>
-  </link> -->
+  </link>-->
 </robot>

File: turtlebot3/turtlebot3_description/urdf/turtlebot3_forklift.gazebo.xacro (robot description, xacro)
@@ -96,35 +96,3 @@
     </plugin>
   </gazebo>
-  <!-- <gazebo reference="base_scan">
-    <material>Gazebo/FlatBlack</material>
-    <sensor type="ray" name="lds_lfcd_sensor">
-      <pose>0 0 0 0 0 0</pose>
-      <visualize>$(arg laser_visual)</visualize>
-      <update_rate>5</update_rate>
-      <ray>
-        <scan>
-          <horizontal>
-            <samples>360</samples>
-            <resolution>1</resolution>
-            <min_angle>0.0</min_angle>
-            <max_angle>6.28319</max_angle>
-          </horizontal>
-        </scan>
-        <range>
-          <min>0.120</min>
-          <max>3.5</max>
-          <resolution>0.015</resolution>
-        </range>
-        <noise>
-          <type>gaussian</type>
-          <mean>0.0</mean>
-          <stddev>0.01</stddev>
-        </noise>
-      </ray>
-      <plugin name="gazebo_ros_lds_lfcd_controller" filename="libgazebo_ros_laser.so">
-        <topicName>scan</topicName>
-        <frameName>base_scan</frameName>
-      </plugin>
-    </sensor>
-  </gazebo> -->
 </robot>

File: turtlebot3/turtlebot3_description/urdf/turtlebot3_forklift.urdf.xacro (robot description, xacro)
@@ -140,30 +140,3 @@
   </joint>
   <link name="imu_link"/>
-  <!-- <joint name="scan_joint" type="fixed">
-    <parent link="base_link_forklift"/>
-    <child link="base_scan"/>
-    <origin xyz="-0.032 0 0.172" rpy="0 0 0"/>
-  </joint>
-  <link name="base_scan">
-    <visual>
-      <origin xyz="0 0 0.0" rpy="0 0 0"/>
-      <geometry>
-        <mesh filename="package://turtlebot3_description/meshes/sensors/lds.stl" scale="0.001 0.001 0.001"/>
-      </geometry>
-      <material name="dark"/>
-    </visual>
-    <collision>
-      <origin xyz="0.015 0 -0.0065" rpy="0 0 0"/>
-      <geometry>
-        <cylinder length="0.0315" radius="0.055"/>
-      </geometry>
-    </collision>
-    <inertial>
-      <mass value="0.114" />
-      <origin xyz="0 0 0" />
-      <inertia ixx="0.001" ixy="0.0" ixz="0.0"
-               iyy="0.001" iyz="0.0"
-               izz="0.001" />
-    </inertial>
-  </link> -->
 </robot>

File: turtlebot3/turtlebot3_description/urdf/turtlebot3_forklift_w_load.urdf.xacro (robot description, xacro)
@@ -29,34 +29,4 @@
     </inertial>
   </link>
-<!--
-  <link name="base_fork">
-			<inertial>
-				<origin xyz="0 0 0" rpy="0 0 0" />
-				<mass value="0.01"/>
-				<inertia ixx="0.01" ixy="0" ixz="0" iyy="0.01" iyz="0" izz="0.01" />
-			</inertial>
-			<visual>
-				<origin xyz="-0.5 0 0" rpy="0 0 0" />
-				<geometry>
-					<mesh filename="package://turtlebot3_description/meshes/bases/forklift_fork.STL" scale="3.0 3.0 3.0"/>
-				</geometry>
-				<material name="grey" />
-			</visual>
-			<collision>
-				<origin xyz="-1 0 0" rpy="0 0 0" />
-				<geometry>
-					<mesh filename="package://turtlebot3_description/meshes/bases/forklift_fork.STL"/>
-				</geometry>
-			</collision>
-		</link>
-		<joint name="fork_axis" type="prismatic">
-			<origin xyz="0 0 -0.14" rpy="0 0 0" />
-			<parent link="base_link_forklift"/>
-			<child link="base_fork"/>
-			<axis xyz="0 0 1" />
-			<dynamics damping="1.0" friction="1.0" />
-			<limit effort="1" velocity="0.2" lower="0" upper="0.2"/>
-    	<safety_controller k_position="20" k_velocity="25" soft_lower_limit="-0.1" soft_upper_limit="0.2" />
-		</joint> -->
   <joint name="wheel_left_joint" type="continuous">
     <parent link="base_link_forklift"/>
@@ -141,30 +111,3 @@
   </joint>
   <link name="imu_link"/>
-  <!-- <joint name="scan_joint" type="fixed">
-    <parent link="base_link_forklift"/>
-    <child link="base_scan"/>
-    <origin xyz="-0.032 0 0.172" rpy="0 0 0"/>
-  </joint>
-  <link name="base_scan">
-    <visual>
-      <origin xyz="0 0 0.0" rpy="0 0 0"/>
-      <geometry>
-        <mesh filename="package://turtlebot3_description/meshes/sensors/lds.stl" scale="0.001 0.001 0.001"/>
-      </geometry>
-      <material name="dark"/>
-    </visual>
-    <collision>
-      <origin xyz="0.015 0 -0.0065" rpy="0 0 0"/>
-      <geometry>
-        <cylinder length="0.0315" radius="0.055"/>
-      </geometry>
-    </collision>
-    <inertial>
-      <mass value="0.114" />
-      <origin xyz="0 0 0" />
-      <inertia ixx="0.001" ixy="0.0" ixz="0.0"
-               iyy="0.001" iyz="0.0"
-               izz="0.001" />
-    </inertial>
-  </link> -->
 </robot>

File: turtlebot3/turtlebot3_description/urdf/turtlebot3_waffle.gazebo.xacro (robot description, xacro)
@@ -102,5 +102,5 @@
     </plugin>
   </gazebo>
-  <!-- <gazebo reference="base_scan">
+  <gazebo reference="base_scan">
     <material>Gazebo/FlatBlack</material>
     <sensor type="ray" name="lds_lfcd_sensor">
@@ -176,4 +176,4 @@
       </plugin>
     </sensor>
-  </gazebo> -->
+  </gazebo>
 </robot>

File: turtlebot3/turtlebot3_description/urdf/turtlebot3_waffle.urdf.xacro (robot description, xacro)
@@ -137,10 +137,10 @@
   </joint>
   <link name="imu_link"/>
-  <!-- <joint name="scan_joint" type="fixed">
+  <joint name="scan_joint" type="fixed">
     <parent link="base_link"/>
     <child link="base_scan"/>
     <origin xyz="-0.064 0 0.122" rpy="0 0 0"/>
-  </joint> -->
-  <!-- <link name="base_scan">
+  </joint>
+  <link name="base_scan">
     <visual>
       <origin xyz="0 0 0" rpy="0 0 0"/>
@@ -163,6 +163,6 @@
                izz="0.001" />
     </inertial>
-  </link> -->
-  <!-- <joint name="camera_joint" type="fixed">
+  </link>
+  <joint name="camera_joint" type="fixed">
     <origin xyz="0.064 -0.065 0.094" rpy="0 0 0"/>
     <parent link="base_link"/>
@@ -181,7 +181,7 @@
         <box size="0.012 0.132 0.020"/>
       </geometry>
-    </collision> -->
+    </collision>
     <!-- This inertial field needs doesn't contain reliable data!! -->
-<!--   <inertial>
+  <inertial>
       <mass value="0.564" />
       <origin xyz="0 0 0" />
@@ -189,6 +189,6 @@
                iyy="0.000498940" iyz="0.0"
                izz="0.003879257" />
-    </inertial>-->
-  <!-- </link>
+    </inertial>
+  </link>
   <joint name="camera_rgb_joint" type="fixed">
     <origin xyz="${r200_cam_rgb_px} ${r200_cam_rgb_py} ${r200_cam_rgb_pz}" rpy="0 0 0"/>
@@ -214,4 +214,4 @@
     <child link="camera_depth_optical_frame"/>
   </joint>
-  <link name="camera_depth_optical_frame"/> -->
+  <link name="camera_depth_optical_frame"/>
 </robot>
