Commit message: clear miscellaneous

File: turtlebot3/turtlebot3_description/urdf/turtlebot3_waffle_w_load.gazebo.xacro (robot description, xacro)
@@ -1,7 +1,8 @@
 <?xml version="1.0"?>
-<robot name="turtlebot3_burger_sim" xmlns:xacro="http://ros.org/wiki/xacro">
-  <xacro:arg name="laser_visual" default="false"/>
-  <xacro:arg name="imu_visual"   default="false"/>
-  <gazebo reference="base_link_burger">
+<robot name="turtlebot3_waffle_sim" xmlns:xacro="http://ros.org/wiki/xacro">
+  <xacro:arg name="laser_visual"  default="false"/>
+  <xacro:arg name="camera_visual" default="false"/>
+  <xacro:arg name="imu_visual"    default="false"/>
+  <gazebo reference="base_link">
     <material>Gazebo/DarkGrey</material>
   </gazebo>
@@ -26,5 +27,14 @@
     <material>Gazebo/FlatBlack</material>
   </gazebo>
-  <gazebo reference="caster_back_link">
+  <gazebo reference="caster_back_right_link">
+    <mu1>0.1</mu1>
+    <mu2>0.1</mu2>
+    <kp>1000000.0</kp>
+    <kd>100.0</kd>
+    <minDepth>0.001</minDepth>
+    <maxVel>1.0</maxVel>
+    <material>Gazebo/FlatBlack</material>
+  </gazebo>
+  <gazebo reference="caster_back_left_link">
     <mu1>0.1</mu1>
     <mu2>0.1</mu2>
@@ -40,8 +50,8 @@
       <visualize>$(arg imu_visual)</visualize>
     </sensor>
-    <material>Gazebo/FlatBlack</material>
+    <material>Gazebo/Grey</material>
   </gazebo>
   <gazebo>
-    <plugin name="turtlebot3_burger_controller" filename="libgazebo_ros_diff_drive.so">
+    <plugin name="turtlebot3_waffle_controller" filename="libgazebo_ros_diff_drive.so">
       <commandTopic>cmd_vel</commandTopic>
       <odometryTopic>odom</odometryTopic>
@@ -49,5 +59,5 @@
       <odometrySource>world</odometrySource>
       <publishOdomTF>true</publishOdomTF>
-      <robotBaseFrame>base_footprint_burger</robotBaseFrame>
+      <robotBaseFrame>base_footprint</robotBaseFrame>
       <publishWheelTF>false</publishWheelTF>
       <publishTf>true</publishTf>
@@ -57,5 +67,5 @@
       <leftJoint>wheel_left_joint</leftJoint>
       <rightJoint>wheel_right_joint</rightJoint>
-      <wheelSeparation>0.160</wheelSeparation>
+      <wheelSeparation>0.287</wheelSeparation>
       <wheelDiameter>0.066</wheelDiameter>
       <wheelAcceleration>1</wheelAcceleration>
@@ -92,4 +102,5 @@
     </plugin>
   </gazebo>
+<!--
   <gazebo reference="base_scan">
     <material>Gazebo/FlatBlack</material>
@@ -124,3 +135,46 @@
     </sensor>
   </gazebo>
+  <gazebo reference="camera_rgb_frame">
+    <sensor type="depth" name="realsense_R200">
+      <always_on>true</always_on>
+      <visualize>$(arg camera_visual)</visualize>
+      <camera>
+          <horizontal_fov>1.3439</horizontal_fov>
+          <image>
+              <width>1920</width>
+              <height>1080</height>
+              <format>R8G8B8</format>
+          </image>
+          <depth_camera></depth_camera>
+          <clip>
+              <near>0.03</near>
+              <far>100</far>
+          </clip>
+      </camera>
+      <plugin name="camera_controller" filename="libgazebo_ros_openni_kinect.so">
+        <baseline>0.2</baseline>
+        <alwaysOn>true</alwaysOn>
+        <updateRate>30.0</updateRate>
+        <cameraName>camera</cameraName>
+        <frameName>camera_rgb_optical_frame</frameName>
+        <imageTopicName>rgb/image_raw</imageTopicName>
+        <depthImageTopicName>depth/image_raw</depthImageTopicName>
+        <pointCloudTopicName>depth/points</pointCloudTopicName>
+        <cameraInfoTopicName>rgb/camera_info</cameraInfoTopicName>
+        <depthImageCameraInfoTopicName>depth/camera_info</depthImageCameraInfoTopicName>
+        <pointCloudCutoff>0.4</pointCloudCutoff>
+            <hackBaseline>0.07</hackBaseline>
+            <distortionK1>0.0</distortionK1>
+            <distortionK2>0.0</distortionK2>
+            <distortionK3>0.0</distortionK3>
+            <distortionT1>0.0</distortionT1>
+            <distortionT2>0.0</distortionT2>
+        <CxPrime>0.0</CxPrime>
+        <Cx>0.0</Cx>
+        <Cy>0.0</Cy>
+        <focalLength>0</focalLength>
+        <hackBaseline>0</hackBaseline>
+      </plugin>
+    </sensor>
+  </gazebo> -->
 </robot>

File: turtlebot3/turtlebot3_description/urdf/turtlebot3_waffle_w_load.urdf.xacro (robot description, xacro)
@@ -2,5 +2,5 @@
 <robot name="turtlebot3_waffle" xmlns:xacro="http://ros.org/wiki/xacro">
   <xacro:include filename="$(find turtlebot3_description)/urdf/common_properties.xacro"/>
-  <xacro:include filename="$(find turtlebot3_description)/urdf/turtlebot3_waffle.gazebo.xacro"/>
+  <xacro:include filename="$(find turtlebot3_description)/urdf/turtlebot3_waffle_w_load.gazebo.xacro"/>
   <xacro:property name="r200_cam_rgb_px" value="0.005"/>
   <xacro:property name="r200_cam_rgb_py" value="0.018"/>
@@ -141,6 +141,6 @@
     <child link="base_scan"/>
     <origin xyz="-0.064 0 0.122" rpy="0 0 0"/>
-  </joint> -->
-  <!-- <link name="base_scan">
+  </joint>
+  <link name="base_scan">
     <visual>
       <origin xyz="0 0 0" rpy="0 0 0"/>
@@ -163,6 +163,6 @@
                izz="0.001" />
     </inertial>
-  </link> -->
-  <!-- <joint name="camera_joint" type="fixed">
+  </link>
+  <joint name="camera_joint" type="fixed">
     <origin xyz="0.064 -0.065 0.094" rpy="0 0 0"/>
     <parent link="base_link"/>
@@ -181,7 +181,6 @@
         <box size="0.012 0.132 0.020"/>
       </geometry>
-    </collision> -->
-    <!-- This inertial field needs doesn't contain reliable data!! -->
-<!--   <inertial>
+    </collision>
+  <inertial>
       <mass value="0.564" />
       <origin xyz="0 0 0" />
@@ -189,6 +188,6 @@
                iyy="0.000498940" iyz="0.0"
                izz="0.003879257" />
-    </inertial>-->
-  <!-- </link>
+    </inertial>
+  </link>
   <joint name="camera_rgb_joint" type="fixed">
     <origin xyz="${r200_cam_rgb_px} ${r200_cam_rgb_py} ${r200_cam_rgb_pz}" rpy="0 0 0"/>

Commit message: edit amr collisiona and visual position

File: turtlebot3/turtlebot3_description/urdf/amr.urdf.xacro (robot description, xacro)
@@ -11,5 +11,5 @@
   <link name="base_link">
     <visual>
-      <origin xyz="-0.032 0 0.0" rpy="0 0 0"/>
+      <origin xyz="-0.032 0 0.050" rpy="0 0 0"/>
       <geometry>
         <mesh filename="package://turtlebot3_description/meshes/bases/robot_base.dae" scale="0.5 0.5 0.3"/>
@@ -18,7 +18,7 @@
     </visual>
     <collision>
-      <origin xyz="-0.032 0 0.250" rpy="0 0 0"/>
+      <origin xyz="-0.032 0 0.10" rpy="0 0 0"/>
       <geometry>
-        <mesh filename="package://turtlebot3_description/meshes/bases/robot_base.dae" scale="0.5 0.7 0.3"/>
+        <mesh filename="package://turtlebot3_description/meshes/bases/robot_base.dae" scale="0.5 0.5 0.3"/>
       </geometry>
     </collision>

File: turtlebot3/turtlebot3_description/urdf/amr_w_load.urdf.xacro (robot description, xacro)
@@ -11,5 +11,5 @@
   <link name="base_link">
     <visual>
-      <origin xyz="-0.032 0 0.0" rpy="0 0 0"/>
+      <origin xyz="-0.032 0 0.050" rpy="0 0 0"/>
       <geometry>
         <mesh filename="package://turtlebot3_description/meshes/bases/robot_base_w_load.dae" scale="0.5 0.5 0.7"/>
@@ -20,5 +20,5 @@
       <origin xyz="-0.032 0 0.250" rpy="0 0 0"/>
       <geometry>
-        <mesh filename="package://turtlebot3_description/meshes/bases/robot_base_w_load.dae" scale="0.5 0.7 0.7"/>
+        <mesh filename="package://turtlebot3_description/meshes/bases/robot_base_w_load.dae" scale="0.5 0.5 0.7"/>
       </geometry>
     </collision>

File: turtlebot3/turtlebot3_description/urdf/rectangle_amr.urdf.xacro (robot description, xacro)
@@ -11,5 +11,5 @@
   <link name="base_link">
     <visual>
-      <origin xyz="-0.032 0 0.0" rpy="0 0 0"/>
+      <origin xyz="-0.032 0 0.050" rpy="0 0 0"/>
       <geometry>
         <mesh filename="package://turtlebot3_description/meshes/bases/robot_base.dae" scale="0.5 0.7 0.3"/>
@@ -18,5 +18,5 @@
     </visual>
     <collision>
-      <origin xyz="-0.032 0 0.250" rpy="0 0 0"/>
+      <origin xyz="-0.032 0 0.10" rpy="0 0 0"/>
       <geometry>
         <mesh filename="package://turtlebot3_description/meshes/bases/robot_base.dae" scale="0.5 0.7 0.3"/>

File: turtlebot3/turtlebot3_description/urdf/rectangle_amr_w_load.urdf.xacro (robot description, xacro)
@@ -11,5 +11,5 @@
   <link name="base_link">
     <visual>
-      <origin xyz="-0.032 0 0.0" rpy="0 0 0"/>
+      <origin xyz="-0.032 0 0.050" rpy="0 0 0"/>
       <geometry>
         <mesh filename="package://turtlebot3_description/meshes/bases/robot_base_w_load.dae" scale="0.5 0.7 0.7"/>

File: velodyne_simulator/velodyne_description/urdf/velodyne_warehouse_2.urdf.xacro (robot description, xacro)
@@ -11,15 +11,15 @@
    <parent link="base_footprint" />
     <child link="base_link" />
-    <origin xyz="0 0 0.03" rpy="0 0 0" />
+    <origin xyz="0 0 0.1" rpy="0 0 0" />
   </joint>
   <link name="base_link" >
     <visual>
       <geometry>
-        <box size="60 100 0.03" />
+        <box size="60 100 0.1" />
       </geometry>
     </visual>
     <collision>
       <geometry>
-        <box size="60 100 0.03" />
+        <box size="60 100 0.1" />
       </geometry>
     </collision>
