Commit message: add two new worlds and human, and make all the sensors static

File: velodyne_simulator/velodyne_description/urdf/velodyne_2.urdf.xacro (robot description, xacro)
@@ -16,10 +16,10 @@
     <visual>
       <geometry>
-        <box size="13.6 20.4 0.03" />
+        <box size="60 100 0.03" />
       </geometry>
     </visual>
     <collision>
       <geometry>
-        <box size="13.6 20.4 0.03" />
+        <box size="60 100 0.03" />
       </geometry>
     </collision>
@@ -34,19 +34,35 @@
     <origin xyz="0 0 0.6" rpy="0 0 0" />
   </xacro:HDL-32E>
+   <xacro:include filename="$(find velodyne_description)/urdf/HDL-32E.urdf.xacro"/>
+  <xacro:HDL-32E parent="base_link" name="velodyne1" topic="/velodyne_pc_1" organize_cloud="${organize_cloud}" hz="10" samples="220" gpu="${gpu}">
+    <origin xyz="0 -27.5 0.6" rpy="0 0 0" />
+  </xacro:HDL-32E>
  <xacro:include filename="$(find velodyne_description)/urdf/HDL-32E.urdf.xacro"/>
   <xacro:HDL-32E parent="base_link" name="velodyne2" topic="/velodyne_pc_2" organize_cloud="${organize_cloud}" hz="10" samples="220" gpu="${gpu}">
-    <origin xyz="5 5 0.6" rpy="1.5708 0 0" />
+    <origin xyz="-27.5 0 0.6" rpy="0 0 0" />
   </xacro:HDL-32E>
    <xacro:include filename="$(find velodyne_description)/urdf/HDL-32E.urdf.xacro"/>
   <xacro:HDL-32E parent="base_link" name="velodyne3" topic="/velodyne_pc_3" organize_cloud="${organize_cloud}" hz="10" samples="220" gpu="${gpu}">
-    <origin xyz="5 -5 0.6" rpy="0 1.5708 0" />
+    <origin xyz="-27.5 -27.5 0.6" rpy="0 0 0" />
   </xacro:HDL-32E>
    <xacro:include filename="$(find velodyne_description)/urdf/HDL-32E.urdf.xacro"/>
   <xacro:HDL-32E parent="base_link" name="velodyne4" topic="/velodyne_pc_4" organize_cloud="${organize_cloud}" hz="10" samples="220" gpu="${gpu}">
-    <origin xyz="-5 5 0.6" rpy="0 0 0" />
+    <origin xyz="-27.5 27.5 0.6" rpy="0 0 0" />
   </xacro:HDL-32E>
    <xacro:include filename="$(find velodyne_description)/urdf/HDL-32E.urdf.xacro"/>
   <xacro:HDL-32E parent="base_link" name="velodyne5" topic="/velodyne_pc_5" organize_cloud="${organize_cloud}" hz="10" samples="220" gpu="${gpu}">
-    <origin xyz="-5 -5 0.6" rpy="0 0 0" />
+    <origin xyz="27.5 -27.5 0.6" rpy="0 0 0" />
+  </xacro:HDL-32E>
+   <xacro:include filename="$(find velodyne_description)/urdf/HDL-32E.urdf.xacro"/>
+  <xacro:HDL-32E parent="base_link" name="velodyne6" topic="/velodyne_pc_6" organize_cloud="${organize_cloud}" hz="10" samples="220" gpu="${gpu}">
+    <origin xyz="0 27.5 0.6" rpy="0 0 0" />
+  </xacro:HDL-32E>
+   <xacro:include filename="$(find velodyne_description)/urdf/HDL-32E.urdf.xacro"/>
+  <xacro:HDL-32E parent="base_link" name="velodyne7" topic="/velodyne_pc_7" organize_cloud="${organize_cloud}" hz="10" samples="220" gpu="${gpu}">
+    <origin xyz="27.5 0 0.6" rpy="0 0 0" />
+  </xacro:HDL-32E>
+     <xacro:include filename="$(find velodyne_description)/urdf/HDL-32E.urdf.xacro"/>
+  <xacro:HDL-32E parent="base_link" name="velodyne8" topic="/velodyne_pc_8" organize_cloud="${organize_cloud}" hz="10" samples="220" gpu="${gpu}">
+    <origin xyz="27.5 27.5 0.6" rpy="0 0 0" />
   </xacro:HDL-32E>
 <gazebo>

File: velodyne_simulator/velodyne_description/urdf/velodyne_3.urdf.xacro (robot description, xacro)
@@ -16,10 +16,10 @@
     <visual>
       <geometry>
-        <box size="13.6 20.4 0.03" />
+        <box size="101 101 0.03" />
       </geometry>
     </visual>
     <collision>
       <geometry>
-        <box size="13.6 20.4 0.03" />
+        <box size="101 101 0.03" />
       </geometry>
     </collision>
@@ -34,19 +34,23 @@
     <origin xyz="0 0 0.6" rpy="0 0 0" />
   </xacro:HDL-32E>
+   <xacro:include filename="$(find velodyne_description)/urdf/HDL-32E.urdf.xacro"/>
+  <xacro:HDL-32E parent="base_link" name="velodyne1" topic="/velodyne_pc_1" organize_cloud="${organize_cloud}" hz="10" samples="220" gpu="${gpu}">
+    <origin xyz="0 -27.5 0.6" rpy="0 0 0" />
+  </xacro:HDL-32E>
  <xacro:include filename="$(find velodyne_description)/urdf/HDL-32E.urdf.xacro"/>
   <xacro:HDL-32E parent="base_link" name="velodyne2" topic="/velodyne_pc_2" organize_cloud="${organize_cloud}" hz="10" samples="220" gpu="${gpu}">
-    <origin xyz="5 5 0.6" rpy="1.5708 0 0" />
+    <origin xyz="-27.5 0 0.6" rpy="0 0 0" />
   </xacro:HDL-32E>
    <xacro:include filename="$(find velodyne_description)/urdf/HDL-32E.urdf.xacro"/>
   <xacro:HDL-32E parent="base_link" name="velodyne3" topic="/velodyne_pc_3" organize_cloud="${organize_cloud}" hz="10" samples="220" gpu="${gpu}">
-    <origin xyz="5 -5 0.6" rpy="0 1.5708 0" />
+    <origin xyz="-27.5 -27.5 0.6" rpy="0 0 0" />
   </xacro:HDL-32E>
    <xacro:include filename="$(find velodyne_description)/urdf/HDL-32E.urdf.xacro"/>
   <xacro:HDL-32E parent="base_link" name="velodyne4" topic="/velodyne_pc_4" organize_cloud="${organize_cloud}" hz="10" samples="220" gpu="${gpu}">
-    <origin xyz="-5 5 0.6" rpy="0 0 0" />
+    <origin xyz="-27.5 27.5 0.6" rpy="0 0 0" />
   </xacro:HDL-32E>
    <xacro:include filename="$(find velodyne_description)/urdf/HDL-32E.urdf.xacro"/>
   <xacro:HDL-32E parent="base_link" name="velodyne5" topic="/velodyne_pc_5" organize_cloud="${organize_cloud}" hz="10" samples="220" gpu="${gpu}">
-    <origin xyz="-5 -5 0.6" rpy="0 0 0" />
+    <origin xyz="27.5 -27.5 0.6" rpy="0 0 0" />
   </xacro:HDL-32E>
 <gazebo>

File: velodyne_simulator/velodyne_description/urdf/velodyne_warehouse_2.urdf.xacro (robot description, xacro)
@@ -16,10 +16,10 @@
     <visual>
       <geometry>
-        <box size="13.6 20.4 0.03" />
+        <box size="60 100 0.03" />
       </geometry>
     </visual>
     <collision>
       <geometry>
-        <box size="13.6 20.4 0.03" />
+        <box size="60 100 0.03" />
       </geometry>
     </collision>

File: velodyne_simulator/velodyne_description/urdf/velodyne_warehouse_3.urdf.xacro (robot description, xacro)
@@ -16,10 +16,10 @@
     <visual>
       <geometry>
-        <box size="13.6 20.4 0.03" />
+        <box size="101 101 0.03" />
       </geometry>
     </visual>
     <collision>
       <geometry>
-        <box size="13.6 20.4 0.03" />
+        <box size="101 101 0.03" />
       </geometry>
     </collision>
